Commit message: Update the cuboid and add a black box

File: drake/examples/kuka_iiwa_arm/models/objects/black_box.urdf (robot description, URDF)
Before this commit: robot simple_cuboid, 1 links, 0 joints
Links:
- link base_link: mass 0.068 -> 0.122; geometry collision box size=0.164 0.054 0.170; collision sphere radius=1e-7
